Commit message: added all the files to simulate the ar markers and cup jig with ar tags

File: jig_description/urdf/ar_2.urdf.xacro (robot description, xacro)
@@ -5,5 +5,5 @@
       <origin rpy="0 0 0" xyz="0 0 0"/>
       <geometry>
-        <mesh filename="package://jig_description/meshes/cup_jig.dae"/>
+        <mesh filename="package://jig_description/meshes/ar_2.dae"/>
         <!-- <box size="1 1 1"/> -->
       </geometry>

File: jig_description/urdf/ar_3.urdf.xacro (robot description, xacro)
@@ -5,5 +5,5 @@
       <origin rpy="0 0 0" xyz="0 0 0"/>
       <geometry>
-        <mesh filename="package://jig_description/meshes/cup_jig.dae"/>
+        <mesh filename="package://jig_description/meshes/ar_3.dae"/>
         <!-- <box size="1 1 1"/> -->
       </geometry>

Commit message: added object collision data

File: jig_description/urdf/ar_2.urdf.xacro (robot description, xacro)
@@ -6,12 +6,12 @@
       <geometry>
         <mesh filename="package://jig_description/meshes/ar_2.dae"/>
-        <!-- <box size="1 1 1"/> -->
       </geometry>
-      <!-- <material>
-        <uri>package://materials/scripts</uri>
-        <uri>package://materials/textures</uri>
-        <name>jig/example</name>
-      </material> -->
     </visual>
+    <collision>
+      <origin xyz="0.0 0.0 0.0" rpy="0.0 0.0 0.0"/>
+      <geometry>
+        <mesh filename="package://jig_description/meshes/ar.stl" scale="1.0"/>
+      </geometry>
+    </collision>
     <inertial>
       <mass value="1" />
@@ -19,26 +19,3 @@
     </inertial>
   </link>
-  <!-- <gazebo reference="jig_base_link">
-    <material>example</material>
-  </gazebo> -->
-  <!-- <joint name="base_ar1" type="fixed">
-    <parent link="jig_base_link"/>
-    <child link="aq1"/>
-    <origin xyz="0 0 0.1"/>
-  </joint>
-  <link name="jig_base_link">
-    <visual>
-      <origin rpy="0 0 0" xyz="0 0 0"/>
-      <geometry>
-        <mesh filename="package://jig_description/meshes/base_plate.stl"/>
-      </geometry>
-      <material name="LightGrey">
-        <color rgba="0.7 0.7 0.7 1.0"/>
-      </material>
-    </visual>
-    <inertial>
-      <mass value="1" />
-      <inertia ixx="1.0" ixy="0.0" ixz="0.0" iyy="1.0" iyz="0.0" izz="1.0" />
-    </inertial>
-  </link> -->
 </robot>

File: jig_description/urdf/ar_3.urdf.xacro (robot description, xacro)
@@ -6,12 +6,12 @@
       <geometry>
         <mesh filename="package://jig_description/meshes/ar_3.dae"/>
-        <!-- <box size="1 1 1"/> -->
       </geometry>
-      <!-- <material>
-        <uri>package://materials/scripts</uri>
-        <uri>package://materials/textures</uri>
-        <name>jig/example</name>
-      </material> -->
     </visual>
+    <collision>
+      <origin rpy="0 0 0" xyz="0 0 0"/>
+      <geometry>
+        <mesh filename="package://jig_description/meshes/ar.stl"/>
+      </geometry>
+    </collision>
     <inertial>
       <mass value="1" />
@@ -19,26 +19,3 @@
     </inertial>
   </link>
-  <!-- <gazebo reference="jig_base_link">
-    <material>example</material>
-  </gazebo> -->
-  <!-- <joint name="base_ar1" type="fixed">
-    <parent link="jig_base_link"/>
-    <child link="aq1"/>
-    <origin xyz="0 0 0.1"/>
-  </joint>
-  <link name="jig_base_link">
-    <visual>
-      <origin rpy="0 0 0" xyz="0 0 0"/>
-      <geometry>
-        <mesh filename="package://jig_description/meshes/base_plate.stl"/>
-      </geometry>
-      <material name="LightGrey">
-        <color rgba="0.7 0.7 0.7 1.0"/>
-      </material>
-    </visual>
-    <inertial>
-      <mass value="1" />
-      <inertia ixx="1.0" ixy="0.0" ixz="0.0" iyy="1.0" iyz="0.0" izz="1.0" />
-    </inertial>
-  </link> -->
 </robot>

File: jig_description/urdf/jig.urdf.xacro (robot description, xacro)
@@ -6,12 +6,12 @@
       <geometry>
         <mesh filename="package://jig_description/meshes/cup_jig.dae"/>
-        <!-- <box size="1 1 1"/> -->
       </geometry>
-      <!-- <material>
-        <uri>package://materials/scripts</uri>
-        <uri>package://materials/textures</uri>
-        <name>jig/example</name>
-      </material> -->
     </visual>
+    <collision>
+      <origin rpy="0 0 0" xyz="0 0 0"/>
+      <geometry>
+        <mesh filename="package://jig_description/meshes/cup_jig.stl"/>
+      </geometry>
+    </collision>
     <inertial>
       <mass value="1" />
@@ -19,26 +19,3 @@
     </inertial>
   </link>
-  <!-- <gazebo reference="jig_base_link">
-    <material>example</material>
-  </gazebo> -->
-  <!-- <joint name="base_ar1" type="fixed">
-    <parent link="jig_base_link"/>
-    <child link="aq1"/>
-    <origin xyz="0 0 0.1"/>
-  </joint>
-  <link name="jig_base_link">
-    <visual>
-      <origin rpy="0 0 0" xyz="0 0 0"/>
-      <geometry>
-        <mesh filename="package://jig_description/meshes/base_plate.stl"/>
-      </geometry>
-      <material name="LightGrey">
-        <color rgba="0.7 0.7 0.7 1.0"/>
-      </material>
-    </visual>
-    <inertial>
-      <mass value="1" />
-      <inertia ixx="1.0" ixy="0.0" ixz="0.0" iyy="1.0" iyz="0.0" izz="1.0" />
-    </inertial>
-  </link> -->
 </robot>

Commit message: PID on and working with gripper

File: jig_description/urdf/ar_2.urdf.xacro (robot description, xacro)
@@ -1,5 +1,5 @@
 <?xml version="1.0"?>
-<robot xmlns:xacro="http://www.ros.org/wiki/xacro" name="jig">
-  <link name="jig_base_link">
+<robot xmlns:xacro="http://www.ros.org/wiki/xacro" name="ar_2">
+  <link name="ar_2__link">
     <visual>
       <origin rpy="0 0 0" xyz="0 0 0"/>
@@ -9,12 +9,12 @@
     </visual>
     <collision>
-      <origin xyz="0.0 0.0 0.0" rpy="0.0 0.0 0.0"/>
+       <origin rpy="0 0 0" xyz="0 0 0"/>
       <geometry>
-        <mesh filename="package://jig_description/meshes/ar.stl" scale="1.0"/>
+        <mesh filename="package://jig_description/meshes/ar_2.dae"/>
       </geometry>
     </collision>
     <inertial>
       <mass value="1" />
-      <inertia ixx="1.0" ixy="0.0" ixz="0.0" iyy="1.0" iyz="0.0" izz="1.0" />
+      <inertia ixx="0.01" ixy="-0.00" ixz="0.0" iyy="0.01" iyz="0.0" izz="0.01" />
     </inertial>
   </link>

File: jig_description/urdf/ar_3.urdf.xacro (robot description, xacro)
@@ -1,5 +1,5 @@
 <?xml version="1.0"?>
-<robot xmlns:xacro="http://www.ros.org/wiki/xacro" name="jig">
-  <link name="jig_base_link">
+<robot xmlns:xacro="http://www.ros.org/wiki/xacro" name="ar_3">
+  <link name="ar_3_link">
     <visual>
       <origin rpy="0 0 0" xyz="0 0 0"/>
@@ -11,10 +11,10 @@
       <origin rpy="0 0 0" xyz="0 0 0"/>
       <geometry>
-        <mesh filename="package://jig_description/meshes/ar.stl"/>
+        <mesh filename="package://jig_description/meshes/ar_3.dae"/>
       </geometry>
     </collision>
     <inertial>
       <mass value="1" />
-      <inertia ixx="1.0" ixy="0.0" ixz="0.0" iyy="1.0" iyz="0.0" izz="1.0" />
+      <inertia ixx="0.01" ixy="-0.00" ixz="0.0" iyy="0.01" iyz="0.0" izz="0.01" />
     </inertial>
   </link>

File: jig_description/urdf/jig.urdf.xacro (robot description, xacro)
@@ -11,10 +11,10 @@
       <origin rpy="0 0 0" xyz="0 0 0"/>
       <geometry>
-        <mesh filename="package://jig_description/meshes/cup_jig.stl"/>
+        <mesh filename="package://jig_description/meshes/cup_jig.dae"/>
       </geometry>
     </collision>
     <inertial>
-      <mass value="1" />
-      <inertia ixx="1.0" ixy="0.0" ixz="0.0" iyy="1.0" iyz="0.0" izz="1.0" />
+      <mass value="0.125" />
+      <inertia ixx="0.01" ixy="-0.00" ixz="0.0" iyy="0.01" iyz="0.0" izz="0.01" />
     </inertial>
   </link>

File: world_sim/camera_urdf/camera.xacro (robot description, xacro)
@@ -1,9 +1,9 @@
 <?xml version="1.0"?>
 <robot xmlns:xacro="http://www.ros.org/wiki/xacro" name="camera">
-  <xacro:include filename="$(find world_sim)/urdf/camera.plugins.xacro" />
+  <xacro:include filename="$(find world_sim)/camera_urdf/camera.plugins.xacro" />
   <xacro:property name="camera_size" value="0.02"/>
   <xacro:property name="camera_origin_x" value="0"/>
   <xacro:property name="camera_origin_y" value="0"/>
-  <xacro:property name="camera_origin_z" value="1"/>
+  <xacro:property name="camera_origin_z" value="2.015"/>
   <xacro:property name="camera_link" value="0.05" /> <!-- Size of square 'camera' box -->
   <link name="world"/>
