Commit message: submodule for robotiq 85 gripper

File: jig_description/urdf/jig.urdf.xacro (robot description, xacro)
@@ -19,3 +19,27 @@
     </inertial>
   </link>
+    <joint name="cup_joint" type="fixed">
+      <parent link="jig_base_link"/>
+      <child link="cup_link"/>
+      <axis xyz="0 0 0"/>
+      <origin rpy="0 0.0 0.0" xyz="0.05490451627 0.03060114443 0.0"/>
+    </joint>
+  <link name="cup_link">
+    <visual>
+      <origin rpy="0 0 0" xyz="0 0 0"/>
+      <geometry>
+        <mesh filename="package://jig_description/meshes/cup.dae"/>
+      </geometry>
+    </visual>
+    <collision>
+      <origin rpy="0 0 0" xyz="0 0 0"/>
+      <geometry>
+        <mesh filename="package://jig_description/meshes/cup.dae"/>
+      </geometry>
+    </collision>
+    <inertial>
+      <mass value="0.125" />
+      <inertia ixx="0.01" ixy="-0.00" ixz="0.0" iyy="0.01" iyz="0.0" izz="0.01" />
+    </inertial>
+  </link>
 </robot>

Commit message: added cup link and mesh for use in model

File: jig_description/urdf/jig.urdf.xacro (robot description, xacro)
@@ -19,3 +19,27 @@
     </inertial>
   </link>
+  <joint name="cup_joint" type="fixed">
+    <axis xyz="0 0 0" />
+    <origin xyz="0.04 0.04 0" rpy="0 0 0"/>
+    <parent link="jig_base_link"/>
+    <child link="cup_link"/>
+  </joint>
+  <link name="cup_link">
+    <visual>
+      <origin rpy="0 0 0" xyz="0 0 0"/>
+      <geometry>
+        <mesh filename="package://jig_description/meshes/cup.dae"/>
+      </geometry>
+    </visual>
+    <collision>
+      <origin rpy="0 0 0" xyz="0 0 0"/>
+      <geometry>
+        <mesh filename="package://jig_description/meshes/cup.stl"/>
+      </geometry>
+    </collision>
+    <inertial>
+      <mass value="1" />
+      <inertia ixx="1.0" ixy="0.0" ixz="0.0" iyy="1.0" iyz="0.0" izz="1.0" />
+    </inertial>
+  </link>
 </robot>

Commit message: fixed typo with collision mesh

File: jig_description/urdf/jig.urdf.xacro (robot description, xacro)
@@ -35,5 +35,5 @@
       <origin rpy="0 0 0" xyz="0 0 0"/>
       <geometry>
-        <mesh filename="package://jig_description/meshes/cup.stl"/>
+        <mesh filename="package://jig_description/meshes/cup.dae"/>
       </geometry>
     </collision>

Commit message: removed cup stuff

File: jig_description/urdf/jig.urdf.xacro (robot description, xacro)
@@ -19,27 +19,3 @@
     </inertial>
   </link>
-    <joint name="cup_joint" type="fixed">
-      <parent link="jig_base_link"/>
-      <child link="cup_link"/>
-      <axis xyz="0 0 0"/>
-      <origin rpy="0 0.0 0.0" xyz="0.05490451627 0.03060114443 0.0"/>
-    </joint>
-  <link name="cup_link">
-    <visual>
-      <origin rpy="0 0 0" xyz="0 0 0"/>
-      <geometry>
-        <mesh filename="package://jig_description/meshes/cup.dae"/>
-      </geometry>
-    </visual>
-    <collision>
-      <origin rpy="0 0 0" xyz="0 0 0"/>
-      <geometry>
-        <mesh filename="package://jig_description/meshes/cup.dae"/>
-      </geometry>
-    </collision>
-    <inertial>
-      <mass value="0.125" />
-      <inertia ixx="0.01" ixy="-0.00" ixz="0.0" iyy="0.01" iyz="0.0" izz="0.01" />
-    </inertial>
-  </link>
 </robot>
